File: DIY_Soldering_Station-eagle/ProMini-connection.sch (EAGLE design)
At the start: 38 parts, among them IC1 LM358N, Q1 IRLZ44Z, Q2 IRLZ44Z, T1 BT136, X1 6ESRM-P, X2 HD44780LCD-1602

Commit message: add some titles to scheme
Parts:
- added R20: 100K, resistor:R-EU_0207/7
- added R21, R22, R23, R24, R25, R26: 10K, resistor:R-EU_0207/7
Connections:
- new net N$53: R21.2, R23.1
- new net N$54: R22.1, R23.2
- new net N$55: R22.2, R24.1
- new net N$56: R24.2, R25.1
- new net N$57: R25.2, R26.1
- new net N$58: R26.2
- net +5V: now also R21.1
- net GND: now also R20.1
- net N$50: now also R20.2
Other:
- note added: "24V to 5V"
- note added: "AC dimmer with zero-cross detecrion"
- note added: "Air sensor OpAmp"
- note added: "Buzzer"
- note added: "Control buttons array"
- note added: "DC-DC (used to power 5V logic over USB)"
- note added: "Heater +"
- note added: "Heater -"
- note added: "Internal switch to disable"
- note added: "Iron sensor OpAmp"
- note added: "Magnet switch +"
- note added: "Sensor +"
- note added: "Sensor -"
- note added: "Soft Iron and Air switch"
- note added: "iron"
Changed lines of the file:
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@@
 <setting verticaltext="up"/>
 </settings>
-<grid distance="0.1" unitdist="inch" unit="inch" style="lines" multiple="1" display="no" altdistance="0.01" altunitdist="inch" altunit="inch"/>
+<grid distance="0.1" unitdist="inch" unit="inch" style="lines" multiple="1" display="yes" altdistance="0.01" altunitdist="inch" altunit="inch"/>
 <layers>
 <layer number="1" name="Top" color="4" fill="11" visible="no" active="no"/>
@@
 <part name="P+9" library="supply1" deviceset="+5V" device=""/>
 <part name="P+10" library="supply1" deviceset="+5V" device=""/>
+<part name="R20" library="resistor" deviceset="R-EU_" device="0207/7" value="100K"/>
+<part name="GND27" library="supply1" deviceset="GND" device=""/>
+<part name="P+11" library="supply1" deviceset="+5V" device=""/>
+<part name="R21" library="resistor" deviceset="R-EU_" device="0207/7" value="10K"/>
+<part name="R22" library="resistor" deviceset="R-EU_" device="0207/7" value="10K"/>
+<part name="R23" library="resistor" deviceset="R-EU_" device="0207/7" value="10K"/>
+<part name="R24" library="resistor" deviceset="R-EU_" device="0207/7" value="10K"/>
+<part name="R25" library="resistor" deviceset="R-EU_" device="0207/7" value="10K"/>
+<part name="R26" library="resistor" deviceset="R-EU_" device="0207/7" value="10K"/>
+<part name="S4" library="switch-omron" deviceset="D-TS" device=""/>
+<part name="S5" library="switch-omron" deviceset="D-TS" device=""/>
+<part name="S6" library="switch-omron" deviceset="D-TS" device=""/>
+<part name="S7" library="switch-omron" deviceset="D-TS" device=""/>
+<part name="S8" library="switch-omron" deviceset="D-TS" device=""/>
+<part name="S9" library="switch-omron" deviceset="D-TS" device=""/>
 </parts>
 <sheets>
@@
 <circle x="149.86" y="-88.9" radius="2.54" width="0.1524" layer="91"/>
 <text x="170.18" y="-119.38" size="1.778" layer="91">Air Grounding</text>
+<text x="0" y="27.94" size="1.778" layer="91">Iron sensor OpAmp</text>
+<text x="10.16" y="-43.18" size="1.778" layer="91">Air sensor OpAmp</text>
+<text x="76.2" y="53.34" size="1.778" layer="91">Buzzer</text>
+<text x="99.06" y="93.98" size="1.778" layer="91">24V to 5V</text>
+<text x="119.38" y="106.68" size="1.778" layer="91">Internal switch to disable </text>
+<text x="119.38" y="104.14" size="1.778" layer="91">DC-DC (used to power 5V logic over USB)</text>
+<text x="182.88" y="99.06" size="1.778" layer="91">Control buttons array</text>
+<text x="231.14" y="55.88" size="1.778" layer="91">Soft Iron and Air switch</text>
+<text x="25.4" y="-93.98" size="1.778" layer="91">AC dimmer with zero-cross detecrion</text>
+<text x="22.86" y="55.88" size="1.778" layer="91">iron</text>
+<text x="40.64" y="66.04" size="1.778" layer="91">Heater +</text>
+<text x="40.64" y="50.8" size="1.778" layer="91">Heater -</text>
+<text x="0" y="63.5" size="1.778" layer="91">Sensor -</text>
+<text x="0" y="45.72" size="1.778" layer="91">Sensor +</text>
+<text x="124.46" y="-114.3" size="1.778" layer="91">Sensor +</text>
+<text x="116.84" y="-101.6" size="1.778" layer="91">Sensor -</text>
+<text x="109.22" y="-91.44" size="1.778" layer="91">Magnet switch +</text>
 </plain>
 <instances>
@@
 <instance part="P+9" gate="1" x="233.68" y="53.34"/>
 <instance part="P+10" gate="1" x="251.46" y="53.34"/>
+<instance part="R20" gate="G$1" x="175.26" y="66.04" rot="R90"/>
+<instance part="GND27" gate="1" x="175.26" y="58.42"/>
+<instance part="P+11" gate="1" x="243.84" y="101.6"/>
+<instance part="R21" gate="G$1" x="236.22" y="91.44" rot="R180"/>
+<instance part="R22" gate="G$1" x="215.9" y="91.44" rot="R180"/>
+<instance part="R23" gate="G$1" x="226.06" y="91.44" rot="R180"/>
+<instance part="R24" gate="G$1" x="205.74" y="91.44" rot="R180"/>
+<instance part="R25" gate="G$1" x="195.58" y="91.44" rot="R180"/>
+<instance part="R26" gate="G$1" x="185.42" y="91.44" rot="R180"/>
+<instance part="S4" gate="G$1" x="190.5" y="81.28"/>
+<instance part="S5" gate="G$1" x="200.66" y="81.28"/>
+<instance part="S6" gate="G$1" x="210.82" y="81.28"/>
+<instance part="S7" gate="G$1" x="220.98" y="81.28"/>
+<instance part="S8" gate="G$1" x="231.14" y="81.28"/>
+<instance part="S9" gate="G$1" x="180.34" y="81.28"/>
 </instances>
 <busses>
@@
 <pinref part="GND26" gate="1" pin="GND"/>
 </segment>
+<segment>
+<pinref part="R20" gate="G$1" pin="1"/>
+<pinref part="GND27" gate="1" pin="GND"/>
+</segment>
 </net>
 <net name="N$2" class="0">
@@
 <wire x1="251.46" y1="40.64" x2="251.46" y2="50.8" width="0.1524" layer="91"/>
 <pinref part="P+10" gate="1" pin="+5V"/>
+</segment>
+<segment>
+<wire x1="243.84" y1="91.44" x2="243.84" y2="99.06" width="0.1524" layer="91"/>
+<pinref part="P+11" gate="1" pin="+5V"/>
+<pinref part="R21" gate="G$1" pin="1"/>
+<wire x1="243.84" y1="91.44" x2="241.3" y2="91.44" width="0.1524" layer="91"/>
 </segment>
 </net>
@@
 <wire x1="165.1" y1="43.18" x2="165.1" y2="48.26" width="0.1524" layer="91"/>
 <wire x1="165.1" y1="53.34" x2="165.1" y2="48.26" width="0.1524" layer="91" curve="-180"/>
-<wire x1="165.1" y1="53.34" x2="165.1" y2="66.04" width="0.1524" layer="91"/>
+<wire x1="165.1" y1="53.34" x2="165.1" y2="71.12" width="0.1524" layer="91"/>
+<wire x1="165.1" y1="71.12" x2="175.26" y2="71.12" width="0.1524" layer="91"/>
+<pinref part="R20" gate="G$1" pin="2"/>
+<wire x1="175.26" y1="71.12" x2="180.34" y2="71.12" width="0.1524" layer="91"/>
+<junction x="175.26" y="71.12"/>
+<wire x1="180.34" y1="71.12" x2="190.5" y2="71.12" width="0.1524" layer="91"/>
+<wire x1="190.5" y1="71.12" x2="200.66" y2="71.12" width="0.1524" layer="91"/>
+<wire x1="200.66" y1="71.12" x2="210.82" y2="71.12" width="0.1524" layer="91"/>
+<wire x1="210.82" y1="71.12" x2="220.98" y2="71.12" width="0.1524" layer="91"/>
+<wire x1="220.98" y1="71.12" x2="231.14" y2="71.12" width="0.1524" layer="91"/>
+<wire x1="231.14" y1="71.12" x2="231.14" y2="76.2" width="0.1524" layer="91"/>
+<wire x1="220.98" y1="76.2" x2="220.98" y2="71.12" width="0.1524" layer="91"/>
+<junction x="220.98" y="71.12"/>
+<wire x1="210.82" y1="76.2" x2="210.82" y2="71.12" width="0.1524" layer="91"/>
+<junction x="210.82" y="71.12"/>
+<wire x1="200.66" y1="76.2" x2="200.66" y2="71.12" width="0.1524" layer="91"/>
+<junction x="200.66" y="71.12"/>
+<wire x1="190.5" y1="76.2" x2="190.5" y2="71.12" width="0.1524" layer="91"/>
+<junction x="190.5" y="71.12"/>
+<wire x1="180.34" y1="76.2" x2="180.34" y2="71.12" width="0.1524" layer="91"/>
+<junction x="180.34" y="71.12"/>
 </segment>
 </net>
@@
 </segment>
 </net>
+<net name="N$53" class="0">
+<segment>
+<pinref part="R21" gate="G$1" pin="2"/>
+<pinref part="R23" gate="G$1" pin="1"/>
+<wire x1="231.14" y1="86.36" x2="231.14" y2="91.44" width="0.1524" layer="91"/>
+<junction x="231.14" y="91.44"/>
+</segment>
+</net>
+<net name="N$54" class="0">
+<segment>
+<pinref part="R23" gate="G$1" pin="2"/>
+<pinref part="R22" gate="G$1" pin="1"/>
+<wire x1="220.98" y1="86.36" x2="220.98" y2="91.44" width="0.1524" layer="91"/>
+<junction x="220.98" y="91.44"/>
+</segment>
+</net>
+<net name="N$55" class="0">
+<segment>
+<pinref part="R22" gate="G$1" pin="2"/>
+<pinref part="R24" gate="G$1" pin="1"/>
+<wire x1="210.82" y1="86.36" x2="210.82" y2="91.44" width="0.1524" layer="91"/>
+<junction x="210.82" y="91.44"/>
+</segment>
+</net>
+<net name="N$56" class="0">
+<segment>
+<pinref part="R24" gate="G$1" pin="2"/>
+<pinref part="R25" gate="G$1" pin="1"/>
+<wire x1="200.66" y1="86.36" x2="200.66" y2="91.44" width="0.1524" layer="91"/>
+<junction x="200.66" y="91.44"/>
+</segment>
+</net>
+<net name="N$57" class="0">
+<segment>
+<pinref part="R25" gate="G$1" pin="2"/>
+<pinref part="R26" gate="G$1" pin="1"/>
+<wire x1="190.5" y1="86.36" x2="190.5" y2="91.44" width="0.1524" layer="91"/>
+<junction x="190.5" y="91.44"/>
+</segment>
+</net>
+<net name="N$58" class="0">
+<segment>
+<pinref part="R26" gate="G$1" pin="2"/>
+<wire x1="180.34" y1="86.36" x2="180.34" y2="91.44" width="0.1524" layer="91"/>
+</segment>
+</net>

Commit message: add some res values and done connecting wires
Parts:
- R21: value 10K -> 1K
- R23: value 10K -> 4.7K
Other:
- note added: "Air"
- note added: "Fan +"
- note added: "Fan -"
- note added: "Fan PWM"
- note added: "Heater ~"
- note added: "Iron PWM"
Changed lines of the file:
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@@
 <part name="GND27" library="supply1" deviceset="GND" device=""/>
 <part name="P+11" library="supply1" deviceset="+5V" device=""/>
-<part name="R21" library="resistor" deviceset="R-EU_" device="0207/7" value="10K"/>
+<part name="R21" library="resistor" deviceset="R-EU_" device="0207/7" value="1K"/>
 <part name="R22" library="resistor" deviceset="R-EU_" device="0207/7" value="10K"/>
-<part name="R23" library="resistor" deviceset="R-EU_" device="0207/7" value="10K"/>
+<part name="R23" library="resistor" deviceset="R-EU_" device="0207/7" value="4.7K"/>
 <part name="R24" library="resistor" deviceset="R-EU_" device="0207/7" value="10K"/>
 <part name="R25" library="resistor" deviceset="R-EU_" device="0207/7" value="10K"/>
@@
 <part name="S8" library="switch-omron" deviceset="D-TS" device=""/>
 <part name="S9" library="switch-omron" deviceset="D-TS" device=""/>
+<part name="P+12" library="supply1" deviceset="+5V" device="" value="+24V"/>
 </parts>
 <sheets>
@@
 <text x="116.84" y="-101.6" size="1.778" layer="91">Sensor -</text>
 <text x="109.22" y="-91.44" size="1.778" layer="91">Magnet switch +</text>
+<text x="147.32" y="-76.2" size="1.778" layer="91">Fan +</text>
+<text x="160.02" y="-83.82" size="1.778" layer="91">Fan -</text>
+<text x="170.18" y="-96.52" size="1.778" layer="91">Heater ~</text>
+<text x="147.32" y="-119.38" size="1.778" layer="91">Heater ~</text>
+<text x="73.66" y="-20.32" size="1.778" layer="91">Fan PWM</text>
+<text x="40.64" y="30.48" size="1.778" layer="91">Iron PWM</text>
+<text x="147.32" y="-106.68" size="1.778" layer="91">Air</text>
 </plain>
 <instances>
@@
 <instance part="GND1" gate="1" x="63.5" y="20.32"/>
 <instance part="GND2" gate="1" x="53.34" y="20.32"/>
-<instance part="P+1" gate="1" x="147.32" y="99.06"/>
+<instance part="P+1" gate="1" x="152.4" y="81.28"/>
 <instance part="GND3" gate="1" x="40.64" y="83.82"/>
 <instance part="GND4" gate="1" x="-5.08" y="53.34"/>
@@
 <instance part="S8" gate="G$1" x="231.14" y="81.28"/>
 <instance part="S9" gate="G$1" x="180.34" y="81.28"/>
+<instance part="P+12" gate="1" x="149.86" y="-78.74"/>
 </instances>
 <busses>
@@
 </segment>
 <segment>
-<pinref part="P+1" gate="1" pin="+5V"/>
-<wire x1="147.32" y1="89.0524" x2="147.32" y2="96.52" width="0.1524" layer="91"/>
-</segment>
-<segment>
 <wire x1="15.24" y1="7.62" x2="15.24" y2="15.24" width="0.1524" layer="91"/>
 <pinref part="P+3" gate="1" pin="+5V"/>
 </segment>
 <segment>
-<wire x1="144.78" y1="78.5876" x2="144.78" y2="48.26" width="0.1524" layer="91"/>
+<wire x1="144.78" y1="78.5876" x2="144.78" y2="73.66" width="0.1524" layer="91"/>
+<wire x1="144.78" y1="73.66" x2="144.78" y2="48.26" width="0.1524" layer="91"/>
 <wire x1="144.78" y1="48.26" x2="149.86" y2="48.26" width="0.1524" layer="91"/>
 <junction x="144.78" y="48.26"/>
@@
 <pinref part="P+4" gate="1" pin="+5V"/>
 <wire x1="144.78" y1="48.26" x2="142.3924" y2="48.26" width="0.1524" layer="91"/>
+<wire x1="144.78" y1="73.66" x2="152.4" y2="73.66" width="0.1524" layer="91"/>
+<junction x="144.78" y="73.66"/>
+<wire x1="152.4" y1="73.66" x2="152.4" y2="78.74" width="0.1524" layer="91"/>
+<pinref part="P+1" gate="1" pin="+5V"/>
 </segment>
 <segment>
@@
 <pinref part="R21" gate="G$1" pin="1"/>
 <wire x1="243.84" y1="91.44" x2="241.3" y2="91.44" width="0.1524" layer="91"/>
+</segment>
+<segment>
+<wire x1="149.86" y1="-86.36" x2="149.86" y2="-81.28" width="0.1524" layer="91"/>
+<pinref part="P+12" gate="1" pin="+5V"/>
 </segment>
 </net>
@@
 <wire x1="93.98" y1="-86.36" x2="93.98" y2="-91.44" width="0.1524" layer="91"/>
 <junction x="93.98" y="-86.36"/>
-<wire x1="93.98" y1="-91.44" x2="96.52" y2="-91.44" width="0.1524" layer="91"/>
+<wire x1="104.14" y1="-129.54" x2="104.14" y2="-91.44" width="0.1524" layer="91"/>
+<wire x1="104.14" y1="-91.44" x2="93.98" y2="-91.44" width="0.1524" layer="91"/>
+<wire x1="157.48" y1="-109.22" x2="157.48" y2="-137.16" width="0.1524" layer="91"/>
+<wire x1="157.48" y1="-137.16" x2="104.14" y2="-137.16" width="0.1524" layer="91"/>
+<wire x1="104.14" y1="-137.16" x2="104.14" y2="-134.62" width="0.1524" layer="91"/>
+<wire x1="104.14" y1="-129.54" x2="104.14" y2="-134.62" width="0.1524" layer="91" curve="-180"/>
+<wire x1="162.56" y1="-99.06" x2="187.96" y2="-99.06" width="0.1524" layer="91"/>
+<wire x1="187.96" y1="-99.06" x2="187.96" y2="-142.24" width="0.1524" layer="91"/>
+<wire x1="187.96" y1="-142.24" x2="99.06" y2="-142.24" width="0.1524" layer="91"/>
+<wire x1="99.06" y1="-142.24" x2="99.06" y2="-134.62" width="0.1524" layer="91"/>
+<wire x1="99.06" y1="-129.54" x2="99.06" y2="-134.62" width="0.1524" layer="91" curve="-180"/>
 </segment>
 </net>
@@
 <wire x1="50.8" y1="-111.76" x2="93.98" y2="-111.76" width="0.1524" layer="91"/>
 <wire x1="93.98" y1="-111.76" x2="93.98" y2="-96.52" width="0.1524" layer="91"/>
-<wire x1="93.98" y1="-96.52" x2="96.52" y2="-96.52" width="0.1524" layer="91"/>
+<wire x1="99.06" y1="-129.54" x2="99.06" y2="-96.52" width="0.1524" layer="91"/>
+<wire x1="99.06" y1="-96.52" x2="93.98" y2="-96.52" width="0.1524" layer="91"/>
 </segment>
 </net>
@@
 <wire x1="50.8" y1="-17.78" x2="50.8" y2="-63.5" width="0.1524" layer="91"/>
 <wire x1="50.8" y1="-63.5" x2="134.62" y2="-63.5" width="0.1524" layer="91"/>
-<wire x1="134.62" y1="-63.5" x2="134.62" y2="-73.66" width="0.1524" layer="91"/>
+<wire x1="134.62" y1="-63.5" x2="134.62" y2="-71.12" width="0.1524" layer="91"/>
+<wire x1="134.62" y1="-71.12" x2="142.24" y2="-71.12" width="0.1524" layer="91"/>
+<wire x1="142.24" y1="-71.12" x2="147.32" y2="-71.12" width="0.1524" layer="91" curve="-180"/>
+<wire x1="147.32" y1="-71.12" x2="157.48" y2="-71.12" width="0.1524" layer="91"/>
+<wire x1="157.48" y1="-71.12" x2="157.48" y2="-88.9" width="0.1524" layer="91"/>
 </segment>
 </net>
@@
 </segment>
 </net>
-<net name="N$43" class="0">
-<segment>
-<pinref part="X2" gate="G$1" pin="DB7"/>
-<wire x1="205.74" y1="-27.94" x2="205.74" y2="50.8" width="0.1524" layer="91"/>
-<wire x1="205.74" y1="50.8" x2="152.5524" y2="50.8" width="0.1524" layer="91"/>
-</segment>
-</net>
 <net name="N$44" class="0">
 <segment>
 <pinref part="U$1" gate="G$1" pin="VCC"/>
 <wire x1="142.0876" y1="48.26" x2="137.16" y2="48.26" width="0.1524" layer="91"/>
-</segment>
-</net>
-<net name="N$48" class="0">
-<segment>
-<wire x1="142.0876" y1="50.8" x2="121.92" y2="50.8" width="0.1524" layer="91"/>
-</segment>
-</net>
-<net name="N$49" class="0">
-<segment>
-<wire x1="142.24" y1="50.8" x2="147.32" y2="50.8" width="0.1524" layer="91" curve="-180"/>
-<wire x1="147.32" y1="50.8" x2="152.4" y2="50.8" width="0.1524" layer="91" curve="-180"/>
 </segment>
 </net>
@@
 </segment>
 </net>
+<net name="N$59" class="0">
+<segment>
+<wire x1="142.24" y1="71.12" x2="127" y2="71.12" width="0.1524" layer="91"/>
+<wire x1="127" y1="71.12" x2="127" y2="58.42" width="0.1524" layer="91"/>
+<wire x1="127" y1="58.42" x2="121.92" y2="58.42" width="0.1524" layer="91"/>
+<wire x1="121.92" y1="58.42" x2="121.92" y2="53.34" width="0.1524" layer="91"/>
+<pinref part="X2" gate="G$1" pin="DB7"/>
+<wire x1="205.74" y1="-27.94" x2="205.74" y2="50.8" width="0.1524" layer="91"/>
+<wire x1="205.74" y1="50.8" x2="157.48" y2="50.8" width="0.1524" layer="91"/>
+<wire x1="157.48" y1="50.8" x2="157.48" y2="71.12" width="0.1524" layer="91"/>
+<wire x1="157.48" y1="71.12" x2="147.32" y2="71.12" width="0.1524" layer="91"/>
+<wire x1="147.32" y1="71.12" x2="142.24" y2="71.12" width="0.1524" layer="91" curve="-180"/>
+</segment>
+</net>
